Commit message: Update inertial properties and joint origin for improved robot dynamics

File: src/simple_robot_with_control.urdf (robot description, URDF)
Before this commit: robot nav_robot, 5 links, 4 joints
Links:
- link base_link: mass 1.0 -> 5.0
- link left_wheel: mass 0.5 -> 1.0
- link right_wheel: mass 0.5 -> 1.0
Joints:
- joint caster_joint: origin xyz=0.1 0 0.05 -> xyz=0.08 0 0.05

Commit message: Update robot inertial properties for improved stability and add multi-room warehouse world model

File: src/simple_robot_with_control.urdf (robot description, URDF)
Before this commit: robot nav_robot, 5 links, 4 joints
Links:
- link base_link: mass 5.0 -> 3.0

Commit message: Adjust wheel joint origins and reduce max wheel acceleration for improved maneuverability

File: src/simple_robot_with_control.urdf (robot description, URDF)
Before this commit: robot nav_robot, 5 links, 4 joints
Joints:
- joint left_wheel_joint: origin xyz=0 0.175 0.1 rpy=0 0 0 -> xyz=-0.1 0.175 0.1 rpy=0 0 0
- joint right_wheel_joint: origin xyz=0 -0.175 0.1 rpy=0 0 0 -> xyz=-0.1 -0.175 0.1 rpy=0 0 0
